Commit message: Rewrite description mesh files for moveit setup assistant in Indigo.

File: phantomx_pincher_arm_description/robots/phantomx_pincher_arm.urdf.xacro (robot description, xacro)
@@ -1,16 +1,24 @@
 <?xml version="1.0"?>
-<robot name="phantomx_pincher_arm" xmlns:xacro="http://www.ros.org/wiki/xacro">
+<robot name="phantomx_pincher_arm" xmlns:xacro="http://ros.org/wiki/xacro">
+    <!-- We can configure joints velocity limit and lower/upper limits
+    to allow access to different operational areas, e.g. left handed vs. right handed robot -->
+    <xacro:property name="joints_vlimit" value="1.571"/>
+    <xacro:property name="pan_llimit" value="-1.74"/>
+    <xacro:property name="pan_ulimit" value="1.74"/>
+    <xacro:property name="shoulder_llimit" value="-1.98"/>
+    <xacro:property name="shoulder_ulimit" value="1.88"/>
+    <xacro:property name="elbow_llimit" value="-1.58"/>
+    <xacro:property name="elbow_ulimit" value="0.59"/>
+    <xacro:property name="wrist_llimit" value="-1.79"/>
+    <xacro:property name="wrist_ulimit" value="1.67"/>
 	<!-- Import URDF xacro model -->
-	<xacro:include filename="$(find phantomx_pincher_arm_description)/urdf/phantomx_pincher_arm.urdf.xacro" />
-	<link name="base_footprint">
-		<visual>
-			<origin xyz="0 0 0" rpy="0 0 0"/>
-			<geometry>
-				<box size="0.001 0.001 0.001" />
-			</geometry>
-		</visual>
-	</link>
-	<xacro:phantomx_pincher_arm prefix="arm_" parent="base_footprint">
+	<xacro:include filename="$(find phantomx_pincher_arm_description)/urdf/phantomx_pincher_arm.xacro" />
+	<link name="base_link"/>
+<!--	<xacro:phantomx_pincher_arm prefix="arm_" parent="base_footprint">
 		<origin xyz="0 0 0" rpy="0 0 0" />
 	</xacro:phantomx_pincher_arm>
+-->
+  <phantomx_pincher_arm parent="base_link" color="Red" gripper_color="Red">
+    <origin xyz="0.145 0.0 0.112"/>
+  </phantomx_pincher_arm>
 </robot>

File: phantomx_pincher_arm_description/urdf/arm_hardware.xacro (robot description, xacro)
@@ -11,6 +11,6 @@
     <link name="${name}_link">
       <!-- TODO: This inertial field needs doesn't contain reliable data!! -->
-      <inertial>
-        <mass value="0.055"/>
+       <inertial>
+       <mass value="0.055"/>
         <origin xyz="0 0 0"/>
         <inertia ixx="0.000017012" ixy="0.0" ixz="0.0"
@@ -18,4 +18,10 @@
                  izz="0.000009483"/>
       </inertial>
+      <!--<inertial>
+        <mass value="6.39321" />
+        <inertia ixx="0.04593" ixy="-0.00259" ixz="-3e-05"
+                 iyy="0.03667" iyz="-0.00031"
+                 izz="0.04858" />
+      </inertial>-->
       <visual>
         <origin xyz="0 0 0" rpy="0 0 0"/>

File: phantomx_pincher_arm_description/urdf/phantomx_pincher_arm.urdf.xacro (robot description, xacro)
@@ -16,8 +16,36 @@
     <xacro:include filename="$(find phantomx_pincher_arm_description)/urdf/phantomx_pincher_arm.xacro"/>
     <!-- As we don't have a base here, add a base_link link as location reference -->
-    <link name="base_link"/>
+    <link name="base_link">
+<!--      <inertial>
+        <mass value="6.39321" />
+        <inertia ixx="0.04593" ixy="-0.00259" ixz="-3e-05"
+                 iyy="0.03667" iyz="-0.00031"
+                 izz="0.04858" />
+      </inertial>
+      <visual>
+        <origin xyz="0 0 0" rpy="0 0 0"/>
+        <geometry>
+          <box size="0.5 0.5 "/>
+        </geometry>
+        <material name="Black"/>
+      </visual>
+      <collision>
+        <origin xyz="0 0 0" rpy="0 0 0"/>
+        <geometry>
+          <box size="0.5 0.5 "/>
+        </geometry>
+      </collision> -->
+    </link>
     <!-- phantomx_pincher_arm macro //joints_vlimit="${joints_vlimit}" pan_llimit="-2.617" pan_ulimit="2.617// -->
     <phantomx_pincher_arm parent="base_link" color="White" gripper_color="White">
-        <origin xyz="0.12 0.00 0.140"/>
+        <origin xyz="0.0 0.00 0.0"/>
+<!--        <origin xyz="0.12 0.00 0.140"/-->
     </phantomx_pincher_arm>
+  <!-- ros_control plugin -->
+  <gazebo>
+    <plugin name="gazebo_ros_control" filename="libgazebo_ros_control.so">
+      <robotNamespace>/phantomx_pincher_arm</robotNamespace>
+      <robotSimType>gazebo_ros_control/DefaultRobotHWSim</robotSimType>
+    </plugin>
+  </gazebo>
 </robot>

File: phantomx_pincher_arm_description/urdf/phantomx_pincher_arm.xacro (robot description, xacro)
@@ -68,15 +68,48 @@
       </actuator>
     </transmission>
-  <!-- gripper -->
+  <!-- gripper   -->
   <xacro:include filename="$(find phantomx_pincher_arm_description)/urdf/phantomx_pincher_gripper.xacro"/>
+<!--
+    <link name="arm_wrist_flex_pan_link"/>
+    <joint name="arm_wrist_flex_pan_joint" type="fixed">
+      <origin xyz="0.110 0.0 0.0" rpy="0 0 0"/>
+      <parent link="arm_wrist_flex_link"/>
+      <child link="arm_wrist_flex_pan_link"/>
+      <xacro:insert_block name="origin"/>
+    </joint>
+    <gazebo reference="arm_wrist_flex_pan_link">
+      <material>Gazebo/White</material>
+      <gravity>true</gravity>
+    </gazebo>
+  -->
 <!-- gripper_link -->
-    <link name="gripper_link"/>
+    <link name="gripper_link">
+      <inertial>
+        <mass value="0.0001"/>
+        <origin xyz="0 0 0"/>
+        <inertia ixx="0.0001" ixy="0.0" ixz="0.0"
+                 iyy="0.0001" iyz="0.0"
+                 izz="0.0001"/>
+      </inertial>
+    </link>
     <joint name="gripper_link_joint" type="revolute">
       <origin xyz="0.110 0 0" rpy="0 0 0"/>
+      <!--<origin xyz="0.110 0 0" rpy="0 0 0"/-->
       <parent link="arm_wrist_flex_link"/>
+      <!--<parent link="arm_wrist_flex_link"/-->
       <child link="gripper_link"/>
       <limit effort="6" velocity="1" lower="-3.14" upper="3.14"/>
+      <dynamics friction="0.13"/>
       <axis xyz="1 0 0"/>
     </joint>
+    <transmission name="gripper_link_transmission">
+      <type>transmission_interface/SimpleTransmission</type>
+      <joint name="gripper_link_joint" >
+        <hardwareInterface>EffortJointInterface</hardwareInterface>
+      </joint>
+      <actuator name="gripper_link_actuator">
+        <hardwareInterface>EffortJointInterface</hardwareInterface>
+      </actuator>
+    </transmission>
   <!--gazebo>
       <gripper name="gripper">

File: phantomx_pincher_arm_description/urdf/phantomx_pincher_gripper.xacro (robot description, xacro)
@@ -7,18 +7,27 @@
       <origin xyz="0.070 0 0" rpy="0 0 0"/>
       <axis xyz="0 1 0"/>
-      <limit effort="30" velocity="0.5" lower="0.002" upper="0.032"/>
+      <limit effort="30" velocity="0.001" lower="0.002" upper="0.032"/>
       <parent link="arm_wrist_flex_link"/>
       <child link="gripper_active_link"/>
     </joint>
+    <transmission name="gripper_link_transmission">
+      <type>transmission_interface/SimpleTransmission</type>
+      <joint name="gripper_joint" >
+        <hardwareInterface>EffortJointInterface</hardwareInterface>
+      </joint>
+      <actuator name="gripper_actuator">
+        <hardwareInterface>EffortJointInterface</hardwareInterface>
+      </actuator>
+    </transmission>
     <pincher_finger name="gripper_active" color="${color}" >
       <origin xyz="0 0 0" rpy="0 0 0"/>
     </pincher_finger>
     <!-- Finger 2 -->
-    <!-- Note: currently static but should be a Mimic of Finger 1 -->
+    <!-- Note: currently static but should be a Mimic of Finger 1
     <joint name="gripper2_joint" type="fixed">
       <origin xyz="0.070 -0.016 0" rpy="0 0 0"/>
       <parent link="arm_wrist_flex_link"/>
       <child link="gripper_active2_link"/>
-    </joint>
+    </joint>   -->
     <pincher_finger name="gripper_active2" color="${color}" >
       <origin xyz="0 0 0" rpy="${M_PI} 0 0"/>
@@ -26,5 +35,5 @@
     <!-- Using Mimic -->
     <!-- gripper 2 joint -->
-    <!--  TODO: Test Mimic ->
+    <!--  TODO: Test Mimic -->
     <joint name="gripper2_joint" type="prismatic">
       <origin xyz="0.070 0 0" rpy="0 0 0"/>
@@ -33,5 +42,14 @@
       <parent link="arm_wrist_flex_link"/>
       <child link="gripper_active2_link"/>
-      <mimic joint="gripper_joint" multiplier="-1"  offset = "0"/>
-    </joint-->
+<!--      <mimic joint="gripper_joint" multiplier="-1"  offset = "0"/-->
+    </joint>
+    <transmission name="gripper2_link_transmission">
+      <type>transmission_interface/SimpleTransmission</type>
+      <joint name="gripper2_joint" >
+        <hardwareInterface>EffortJointInterface</hardwareInterface>
+      </joint>
+      <actuator name="gripper2_actuator">
+        <hardwareInterface>EffortJointInterface</hardwareInterface>
+      </actuator>
+    </transmission>
 </robot>
