Commit message: Add One Gripper for Gazebo.

File: phantomx_pincher_arm_description/urdf/arm_hardware.xacro (robot description, xacro)
@@ -195,10 +195,15 @@
       <inertial>
         <!-- TODO: This inertial field needs doesn't contain reliable data!! -->
-        <mass value="0.01"/>
-        <origin xyz="0 0 0"/>
-        <inertia ixx="0.000001" ixy="0.0" ixz="0.0"
-                 iyy="0.000001" iyz="0.0"
-                 izz="0.000001"/>
-      </inertial>
+        <origin xyz="0 0 0"/>
+        <!--mass value="0.01"/-->
+        <!--inertia ixx="0.000001" ixy="0.0" ixz="0.0"
+                 iyy="0.000001" iyz="0.0"
+                 izz="0.000001"/-->
+        <mass value="0.00805661848049576" />
+         <!-- Inertial matrix ixx/iyy/izz increased to make gazebo happy -->
+        <inertia ixx="5.11986620594033E-03" ixy="-3.30249741353407E-09" ixz="1.24817528594142E-12"
+               iyy="2.94192770039741E-03" iyz="7.56956725380165E-12"
+               izz="2.63439537656996E-03" />
+        </inertial>
       <visual>
         <xacro:insert_block name="origin"/>

File: phantomx_pincher_arm_description/urdf/phantomx_pincher_gripper.xacro (robot description, xacro)
@@ -7,9 +7,11 @@
       <origin xyz="0.070 0 0" rpy="0 0 0"/>
       <axis xyz="0 1 0"/>
-      <limit effort="30" velocity="0.001" lower="0.002" upper="0.032"/>
+      <dynamics friction="2500"/>
+      <limit effort="30" velocity="0.1" lower="0.002" upper="0.032"/>
       <parent link="arm_wrist_flex_link"/>
       <child link="gripper_active_link"/>
+      <calibration rising="0.0" />
     </joint>
-    <transmission name="gripper_link_transmission">
+    <!--transmission name="gripper_link_transmission">
       <type>transmission_interface/SimpleTransmission</type>
       <joint name="gripper_joint" >
@@ -19,4 +21,16 @@
         <hardwareInterface>EffortJointInterface</hardwareInterface>
       </actuator>
+    </transmission-->
+    <!-- version GripperCommand -->
+    <transmission name="gripper_link_transmission">
+      <type>transmission_interface/SimpleTransmission</type>
+      <joint name="gripper_joint" >
+        <hardwareInterface>EffortJointInterface</hardwareInterface>
+		<mechanicalReduction>1</mechanicalReduction>
+      </joint>
+      <actuator name="gripper_actuator">
+        <hardwareInterface>PositionJointInterface</hardwareInterface>
+		<mechanicalReduction>1</mechanicalReduction>
+      </actuator>
     </transmission>
     <pincher_finger name="gripper_active" color="${color}" >
@@ -24,10 +38,10 @@
     </pincher_finger>
     <!-- Finger 2 -->
-    <!-- Note: currently static but should be a Mimic of Finger 1
+    <!-- Note: currently static but should be a Mimic of Finger 1-->
     <joint name="gripper2_joint" type="fixed">
-      <origin xyz="0.070 -0.016 0" rpy="0 0 0"/>
+      <origin xyz="0.070 -0.006 0" rpy="0 0 0"/>
       <parent link="arm_wrist_flex_link"/>
       <child link="gripper_active2_link"/>
-    </joint>   -->
+    </joint>
     <pincher_finger name="gripper_active2" color="${color}" >
       <origin xyz="0 0 0" rpy="${M_PI} 0 0"/>
@@ -36,13 +50,15 @@
     <!-- gripper 2 joint -->
     <!--  TODO: Test Mimic -->
-    <joint name="gripper2_joint" type="prismatic">
+    <!--joint name="gripper2_joint" type="prismatic">
       <origin xyz="0.070 0 0" rpy="0 0 0"/>
       <axis xyz="0 1 0"/>
-      <limit effort="30" velocity="0.5" lower="-0.016" upper="-0.002"/>
+      <dynamics friction="2500"/>
+      <limit effort="30" velocity="0.1" lower="-0.032" upper="-0.002"/>
       <parent link="arm_wrist_flex_link"/>
       <child link="gripper_active2_link"/>
+      <calibration rising="0.0" /-->
 <!--      <mimic joint="gripper_joint" multiplier="-1"  offset = "0"/-->
-    </joint>
-    <transmission name="gripper2_link_transmission">
+    <!--/joint-->
+    <!--transmission name="gripper2_link_transmission">
       <type>transmission_interface/SimpleTransmission</type>
       <joint name="gripper2_joint" >
@@ -52,4 +68,16 @@
         <hardwareInterface>EffortJointInterface</hardwareInterface>
       </actuator>
-    </transmission>
+    </transmission-->
+    <!-- version GripperCommand
+    <transmission name="gripper2_link_transmission">
+      <type>transmission_interface/SimpleTransmission</type>
+      <joint name="gripper2_joint" >
+        <hardwareInterface>EffortJointInterface</hardwareInterface>
+		<mechanicalReduction>1</mechanicalReduction>
+      </joint>
+      <actuator name="gripper2_actuator">
+        <hardwareInterface>PositionJointInterface</hardwareInterface>
+		<mechanicalReduction>1</mechanicalReduction>
+      </actuator>
+    </transmission>-->
 </robot>

Commit message: Fix one gripper.

File: phantomx_pincher_arm_description/urdf/arm_hardware.xacro (robot description, xacro)
@@ -11,5 +11,5 @@
     <link name="${name}_link">
       <!-- TODO: This inertial field needs doesn't contain reliable data!! -->
-       <inertial>
+       <!--<inertial>
        <mass value="0.055"/>
         <origin xyz="0 0 0"/>
@@ -17,11 +17,11 @@
                  iyy="0.000013258" iyz="0.0"
                  izz="0.000009483"/>
-      </inertial>
-      <!--<inertial>
+      </inertial>-->
+      <inertial>
         <mass value="6.39321" />
         <inertia ixx="0.04593" ixy="-0.00259" ixz="-3e-05"
                  iyy="0.03667" iyz="-0.00031"
                  izz="0.04858" />
-      </inertial>-->
+      </inertial>
       <visual>
         <origin xyz="0 0 0" rpy="0 0 0"/>

File: phantomx_pincher_arm_description/urdf/phantomx_pincher_arm.urdf.xacro (robot description, xacro)
@@ -26,5 +26,5 @@
         <origin xyz="0 0 0" rpy="0 0 0"/>
         <geometry>
-          <box size="0.5 0.5 "/>
+          <box size="0.5 0.5 0.5"/>
         </geometry>
         <material name="Black"/>

File: phantomx_pincher_arm_description/urdf/phantomx_pincher_gripper.xacro (robot description, xacro)
@@ -7,5 +7,5 @@
       <origin xyz="0.070 0 0" rpy="0 0 0"/>
       <axis xyz="0 1 0"/>
-      <dynamics friction="2500"/>
+      <dynamics damping="5.0"/>
       <limit effort="30" velocity="0.1" lower="0.002" upper="0.032"/>
       <parent link="arm_wrist_flex_link"/>
